File: PCB/TOTEM-SHIFT 0.4/TOTEM-SHIFT 0.4.kicad_pcb (KiCad board)
At the start: 2 copper layers, 258.7 x 92.2 mm, 102 parts, among them U1 xiao-ble, U2 xiao-ble

Commit message: Testing Hidden Power Switch
Parts:
- removed BAT+3, BAT+4: +, TOTEMlib:BatteryPad
- removed BATGND3, BATGND4: -, TOTEMlib:BatteryPad
- DL1, DL10, DL11, DL12, DL13, DL14, DL15, DL16, DL17, DL18, DL19, DL2, DL3, DL4, DL5, DL6, DL7, DL8, DL9, DR1, DR10, DR11, DR12, DR13, DR14, DR15, DR16, DR17, DR18, DR19, DR2, DR3, DR4, DR5, DR6, DR7, DR8, DR9: moved to B.Cu
- moved BAT+2 62.6 mm to (165.4, 61.0)
- moved BATGND2 62.6 mm to (160.4, 61.0)
- moved BAT+1 62.2 mm to (134.7, 61.0)
- moved BATGND1 62.2 mm to (139.7, 61.0)
Routing:
- net VBAT_R: track 151.6 -> 91.1 mm
- net VBAT_L: track 147.9 -> 95.3 mm
- net COL1_R: track 84.0 -> 89.7 mm
- net COL2_R: track 175.8 -> 181.2 mm
- net COL2_L: track 143.6 -> 147.3 mm
- net Net-(DL12-A): track 143.0 -> 139.3 mm
- net Net-(DL7-A): track 164.0 -> 160.4 mm
- net ROW0_L: track 227.4 -> 231.0 mm, vias 7 -> 2
- net ROW1_L: track 225.6 -> 229.2 mm, vias 7 -> 2
- net Net-(DL2-A): track 185.1 -> 181.6 mm
- net ROW2_L: track 223.9 -> 227.3 mm, vias 7 -> 2
- net ROW3_L: track 207.4 -> 210.7 mm
- net COL3_R: track 195.0 -> 198.2 mm
- net Net-(DL11-A): track 143.7 -> 140.7 mm
- net COL0_L: track 98.7 -> 101.7 mm
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Other:
- board text removed: "0.1"
- board text removed: "T O T E M"

Commit message: Small PCB trace fixes
Routing:
- net Net-(DL16-A): track 25.9 -> 30.7 mm, vias 2 -> 3
- net COL2_R: track 181.2 -> 177.5 mm
- net ROW3_R: track 205.6 -> 208.0 mm, vias 1 -> 3
- net ROW3_L: track 210.7 -> 212.9 mm, vias 1 -> 3
- net Net-(DR17-A): track 61.2 -> 59.8 mm
- net COL1_R: track 89.7 -> 88.4 mm
- net ROW1_L: track 229.2 -> 230.2 mm
- net ROW1_R: track 240.1 -> 240.8 mm
- net ROW0_R: track 235.6 -> 236.2 mm
- net ROW2_L: track 227.3 -> 227.9 mm
- net Net-(DR15-A): track 64.9 -> 65.1 mm, vias 1 -> 2
- net Net-(DR6-A): track 142.2 -> 142.1 mm, vias 1 -> 2
- net Net-(DL11-A): track 140.7 -> 140.8 mm, vias 1 -> 2
- net Net-(DL12-A): track 139.3 -> 139.4 mm, vias 1 -> 2
- net Net-(DR1-A): track 156.4 -> 156.3 mm, vias 1 -> 2
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
Commit message: Major changes, hidden switches and case redesign
Parts:
- RST (x2): footprint Button_Switch_THT:SW_PUSH_6mm_H5mm -> Button_Switch_THT:SW_PUSH_1P1T_6x3.5mm_H5.0_APEM_MJTP1250
- moved PWR 81.6 mm to (157.2, 50.7), turned to 0 degrees
- moved PWR 74.2 mm to (142.7, 58.5), turned to 180 degrees
- moved RST 6.27 mm to (136.7, 51.4), turned to -90 degrees
- moved BAT+1 2.51 mm to (134.6, 63.5)
- moved BATGND1 2.51 mm to (139.6, 63.5)
- moved BAT+2 2.50 mm to (165.3, 63.5)
- moved BATGND2 2.50 mm to (160.3, 63.5)
- moved RST 0.74 mm to (163.4, 51.4)
Routing:
- net BAT+_R: track 29.9 -> 120.4 mm, vias 1 -> 5
- net BAT+_L: track 36.8 -> 124.7 mm, vias 2 -> 0
- net VBAT_L: track 95.3 -> 17.3 mm, vias 2 -> 0
- net VBAT_R: track 91.1 -> 15.8 mm, vias 4 -> 0
- net COL1_R: track 88.4 -> 101.4 mm
- net Net-(DR19-A): track 43.9 -> 37.9 mm
- net Net-(DL19-A): track 43.7 -> 49.0 mm
- net ROW3_R: track 208.0 -> 212.6 mm, vias 3 -> 4
- net RESET_L: track 134.9 -> 132.3 mm
- net COL4_L: track 211.1 -> 208.6 mm
- net RESET_R: track 136.9 -> 139.2 mm, vias 0 -> 2
- net COL4_R: track 240.7 -> 239.1 mm
- net Net-(DL1-A): track 178.3 -> 176.8 mm
- net COL2_R: track 177.5 -> 178.7 mm
- net GND_R: vias 31 -> 34
Other:
- outline, holes or cut-outs redrawn
