File: PCB/TOTEM-SHIFT 0.4/TOTEM-SHIFT 0.4.kicad_pcb (KiCad board)
At the start: 2 copper layers, 258.7 x 92.2 mm, 98 parts, among them U1 xiao-ble, U2 xiao-ble

Commit message: PCB ready for production update
Parts:
- moved BAT+2 1.01 mm to (165.3, 62.5)
- moved BATGND2 1.01 mm to (160.3, 62.5)
- moved BAT+1 1.01 mm to (134.6, 62.5)
- moved BATGND1 1.01 mm to (139.6, 62.5)
Routing:
- net VBAT_R: track 15.8 -> 14.8 mm
- net VBAT_L: track 17.3 -> 16.3 mm
