File: PCB/TOTEM-SHIFT 0.4/TOTEM-SHIFT 0.4.kicad_sch (KiCad schematic)
At the start: 90 parts, among them U1 xiao-ble, U2 xiao-ble

Commit message: Major changes, hidden switches and case redesign
Parts:
- RSW1, RSW2: footprint Button_Switch_THT:SW_PUSH_6mm_H5mm -> Button_Switch_THT:SW_PUSH_1P1T_6x3.5mm_H5.0_APEM_MJTP1250
Changed lines of the file:
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@@
 			)
 		)
-		(property "Footprint" "Button_Switch_THT:SW_PUSH_6mm_H5mm"
+		(property "Footprint" "Button_Switch_THT:SW_PUSH_1P1T_6x3.5mm_H5.0_APEM_MJTP1250"
 			(at 125.984 73.152 0)
 			(effects
@@
 			)
 		)
-		(property "Footprint" "Button_Switch_THT:SW_PUSH_6mm_H5mm"
+		(property "Footprint" "Button_Switch_THT:SW_PUSH_1P1T_6x3.5mm_H5.0_APEM_MJTP1250"
 			(at 179.324 73.152 0)
 			(effects
